Commit message: [add] Refactor Go2 Configuration and Description for Ignition Fortress
- Removed obsolete launch files: `ign_gazebo.launch.py` and `ign_gazebo.launch copy.py`.
- Updated `package.xml` for `go2_config` and `go2_description` to reflect new maintainer and dependencies.
- Added new world file `default.sdf` for Ignition Gazebo simulation.
- Introduced new configuration files for robot control in `go2_description`.
- Updated Xacro files to enhance robot model parameters and sensor configurations.
- Removed deprecated `robot_mid360.xacro` and adjusted laser and lidar sensor implementations for compatibility with Ignition Gazebo.
- Improved torque parameters in `const.xacro` for better performance.
- Streamlined launch descriptions to focus on essential nodes and parameters.

File: champ/champ_description/urdf/hokuyo_utm30lx.urdf.xacro (robot description, xacro)
@@ -34,10 +34,10 @@
       </xacro:hokuyo_utm30lx_model>
       <gazebo reference="${name}_frame">
-        <sensor type="ray" name="${name}">
+        <sensor type="gpu_lidar" name="${name}">
           <always_on>true</always_on>
           <update_rate>${update_rate}</update_rate>
           <pose>0 0 0 0 0 0</pose>
           <visualize>false</visualize>
-          <ray>
+          <lidar>
             <scan>
               <horizontal>
@@ -58,14 +58,7 @@
               <stddev>0.004</stddev>
             </noise>
-          </ray>
-          <plugin name="gazebo_ros_${name}_controller" filename="libgazebo_ros_ray_sensor.so">
-            <ros>
-              <argument>~/out:=${ros_topic}</argument>
-            </ros>
-            <!-- Set output to sensor_msgs/PointCloud to get same output type as gazebo_ros_block_laser -->
-            <output_type>sensor_msgs/LaserScan</output_type>
-            <!-- <frame_name> ommited, will default to block_laser_link -->
-            <!-- min_intensity instead of hokuyoMinIntensity -->
-            <min_intensity>100.0</min_intensity>
+          </lidar>
+          <plugin filename="ignition-gazebo-sensors-system" name="ignition::gazebo::systems::Sensors">
+            <ignition_frame_id>${name}_frame</ignition_frame_id>
           </plugin>
         </sensor>
@@ -77,9 +70,9 @@
       </xacro:hokuyo_utm30lx_model>
       <gazebo reference="${name}_frame">
-        <sensor type="gpu_ray" name="${name}">
+        <sensor type="gpu_lidar" name="${name}">
           <update_rate>${update_rate}</update_rate>
           <pose>0 0 0 0 0 0</pose>
           <visualize>false</visualize>
-          <ray>
+          <lidar>
             <scan>
               <horizontal>
@@ -100,11 +93,7 @@
               <stddev>0.004</stddev>
             </noise>
-          </ray>
-          <plugin name="gazebo_ros_${name}_controller" filename="libgazebo_ros_ray_sensor.so">
-            <ros>
-              <argument>~/out:=${ros_topic}</argument>
-            </ros>
-            <output_type>sensor_msgs/LaserScan</output_type>
-            <min_intensity>100.0</min_intensity>
+          </lidar>
+          <plugin filename="ignition-gazebo-sensors-system" name="ignition::gazebo::systems::Sensors">
+            <ignition_frame_id>${name}_frame</ignition_frame_id>
           </plugin>
         </sensor>

File: robots/descriptions/go2_description/xacro/const.xacro (robot description, xacro)
@@ -44,13 +44,13 @@
     <xacro:property name="hip_position_min" value="-1.0472"/>
     <xacro:property name="hip_velocity_max" value="30.1"/>
-    <xacro:property name="hip_torque_max" value="23.7"/>
+    <xacro:property name="hip_torque_max" value="80.0"/>
     <xacro:property name="thigh_position_max" value="3.4907"/>
     <xacro:property name="thigh_position_min" value="-1.5708"/>
     <xacro:property name="thigh_velocity_max" value="30.1"/>
-    <xacro:property name="thigh_torque_max" value="23.7"/>
+    <xacro:property name="thigh_torque_max" value="80.0"/>
     <xacro:property name="calf_position_max" value="-0.83776"/>
     <xacro:property name="calf_position_min" value="-2.7227"/>
     <xacro:property name="calf_velocity_max" value="20.06"/>
-    <xacro:property name="calf_torque_max" value="35.55"/>
+    <xacro:property name="calf_torque_max" value="80.0"/>
     <!-- dynamics inertial value -->
     <!-- trunk -->

File: robots/descriptions/go2_description/xacro/gazebo.xacro (robot description, xacro)
@@ -1,35 +1,20 @@
 <?xml version="1.0"?>
 <robot>
+    <!-- Pose publisher plugin for ground truth odometry -->
     <gazebo>
-      <plugin name="p3d_base_controller" filename="libgazebo_ros_p3d.so">
-        <ros>
-            <!-- <remapping>odom:=odom/ground_truth</remapping> -->
-            <remapping>odom:=odom</remapping>
-        </ros>
-        <body_name>base_link</body_name>
-        <frame_name>world</frame_name>
-        <update_rate>10.0</update_rate>
-        <xyz_offset>0 0 0</xyz_offset>
-        <rpy_offset>0 0 0</rpy_offset>
-        <gaussian_noise>0.01</gaussian_noise>
-    </plugin>
-    </gazebo>
-    <gazebo>
-        <plugin
-        filename="libignition-gazebo-pose-publisher-system.so"
-        name="ignition::gazebo::systems::PosePublisher">
-        <publish_link_pose>true</publish_link_pose>
-        <publish_collision_pose>false</publish_collision_pose>
-        <publish_visual_pose>false</publish_visual_pose>
-        <publish_nested_model_pose>false</publish_nested_model_pose>
+        <plugin filename="ignition-gazebo-pose-publisher-system" name="ignition::gazebo::systems::PosePublisher">
+            <publish_link_pose>true</publish_link_pose>
+            <publish_nested_model_pose>true</publish_nested_model_pose>
+            <use_pose_vector_msg>true</use_pose_vector_msg>
+            <update_frequency>10.0</update_frequency>
         </plugin>
     </gazebo>
+    <!-- Ignition ros2_control plugin -->
     <gazebo>
-        <!-- <plugin filename="libgazebo_ros2_control.so" name="gazebo_ros2_control"> -->
-        <!-- <plugin name="gz_ros2_control::GazeboSimROS2ControlPlugin" filename="libgz_ros2_control-system.so"> -->
         <plugin filename="gz_ros2_control-system" name="gz_ros2_control::GazeboSimROS2ControlPlugin">
-            <parameters>$(find go2_description)/config/ros_control.yaml</parameters>
+            <parameters>$(find go2_description)/config/ros_control/ros_control.yaml</parameters>
         </plugin>
     </gazebo>
+    <!-- IMU sensor -->
     <gazebo reference="imu_link">
         <sensor name="imu_sensor" type="imu">
@@ -78,11 +63,5 @@
             </linear_acceleration>
             </imu>
-            <!-- <plugin name="imu_plugin" filename="libgazebo_ros_imu_sensor.so"> -->
-            <plugin filename="gz-sim-imu-system" name="gz::sim::systems::Imu">
-                <ros>
-                    <namespace>imu</namespace>
-                    <remapping>~/out:=data</remapping>
-                </ros>
-                <initial_orientation_as_reference>false</initial_orientation_as_reference>
+            <plugin filename="ignition-gazebo-imu-system" name="ignition::gazebo::systems::Imu">
             </plugin>
         </sensor>

File: robots/descriptions/go2_description/xacro/laser.xacro (robot description, xacro)
@@ -27,10 +27,10 @@
     </link>
     <gazebo reference="front_laser">
-        <sensor name="front_laser_sensor" type="ray">
+        <sensor name="front_laser_sensor" type="gpu_lidar">
             <always_on>true</always_on>
             <visualize>false</visualize>
             <pose>-0.032 0 0.171 0 0 0</pose>
             <update_rate>50</update_rate>
-            <ray>
+            <lidar>
             <scan>
                 <horizontal>
@@ -51,11 +51,7 @@
                 <stddev>0.01</stddev>
             </noise>
-            </ray>
-            <plugin name="gazebo_ros_front_laserscan" filename="libgazebo_ros_ray_sensor.so">
-            <ros>
-                <remapping>~/out:=scan</remapping>
-            </ros>
-            <output_type>sensor_msgs/LaserScan</output_type>
-            <frame_name>front_laser</frame_name>
+            </lidar>
+            <plugin filename="ignition-gazebo-sensors-system" name="ignition::gazebo::systems::Sensors">
+                <ignition_frame_id>front_laser</ignition_frame_id>
             </plugin>
         </sensor>

File: robots/descriptions/go2_description/xacro/leg.xacro (robot description, xacro)
@@ -146,4 +146,18 @@
                     <sphere radius="${foot_radius}"/>
                 </geometry>
+                <surface>
+                    <friction>
+                        <ode>
+                            <mu>1.2</mu>
+                            <mu2>1.2</mu2>
+                        </ode>
+                    </friction>
+                    <contact>
+                        <ode>
+                            <kp>100000</kp>
+                            <kd>100</kd>
+                        </ode>
+                    </contact>
+                </surface>
             </collision>
             <inertial>
@@ -157,5 +171,4 @@
         <ros2_control name="${name}" type="system">
             <hardware>
-                <!-- <plugin>gazebo_ros2_control/GazeboSystem</plugin> -->
                 <plugin>gz_ros2_control/GazeboSimSystem</plugin>
             </hardware>

File: robots/descriptions/go2_description/xacro/velodyne.xacro (robot description, xacro)
@@ -47,11 +47,13 @@
         </visual>
     </link>
-    <!-- Gazebo requires the velodyne_gazebo_plugins package -->
+    <!-- Ignition Gazebo lidar sensor -->
     <gazebo reference="velodyne">
-        <sensor name="velodyne-VLP16" type="ray">
+        <sensor name="velodyne-VLP16" type="gpu_lidar">
         <pose>0 0 0 0 0 0</pose>
         <visualize>false</visualize>
         <update_rate>10</update_rate>
-        <ray>
+        <topic>velodyne_points</topic>
+        <ignition_frame_id>velodyne</ignition_frame_id>
+        <lidar>
             <scan>
             <horizontal>
@@ -76,18 +78,7 @@
             <type>gaussian</type>
             <mean>0.0</mean>
-            <stddev>0.0</stddev>
+            <stddev>0.008</stddev>
             </noise>
-        </ray>
-        <plugin filename="libgazebo_ros_velodyne_laser.so" name="gazebo_ros_laser_controller">
-            <ros>
-              <namespace>/</namespace>
-              <remapping>~/out:=velodyne_points</remapping>
-            </ros>
-            <frame_name>velodyne</frame_name>
-            <organize_cloud>false</organize_cloud>
-            <min_range>0.9</min_range>
-            <max_range>130.0</max_range>
-            <gaussian_noise>0.008</gaussian_noise>
-        </plugin>
+        </lidar>
         </sensor>
     </gazebo>
